File: Ana/Ana.kicad_pcb (KiCad board)
At the start: 2 copper layers, 68.6 x 53.3 mm, 11 parts, among them J1 Conn_01x02_Female, P1 Power, P2 Analog, P3 Digital, P4 Digital, P5 CONN_01X01, P6 CONN_01X01, P7 CONN_01X01, P8 CONN_01X01

Commit message: Waiting for PCB layout
Parts:
- added C1: 100n, Capacitor_THT:C_Radial_D5.0mm_H7.0mm_P2.00mm, F.Cu at (140.2, 83.2)
- added C2: 100n, Capacitor_THT:C_Radial_D5.0mm_H7.0mm_P2.00mm, F.Cu at (159.3, 109.9)
- added C3: 1u, Capacitor_THT:C_Radial_D5.0mm_H7.0mm_P2.00mm, F.Cu at (141.5, 94.6)
- added C4: 100n, Capacitor_THT:C_Radial_D5.0mm_H7.0mm_P2.00mm, F.Cu at (168.1, 109.9)
- added R1: 10k, Resistor_THT:R_Axial_DIN0207_L6.3mm_D2.5mm_P10.16mm_Horizontal, F.Cu at (125.0, 83.2)
- added R2: 100k, Resistor_THT:R_Axial_DIN0207_L6.3mm_D2.5mm_P10.16mm_Horizontal, F.Cu at (125.0, 89.5)
- added R3: 1k, Resistor_THT:R_Axial_DIN0207_L6.3mm_D2.5mm_P10.16mm_Horizontal, F.Cu at (125.0, 95.9)
- added R4: 100k, Resistor_THT:R_Axial_DIN0207_L6.3mm_D2.5mm_P10.16mm_Horizontal, F.Cu at (125.0, 102.2)
- added R5: 1k, Resistor_THT:R_Axial_DIN0207_L6.3mm_D2.5mm_P10.16mm_Horizontal, F.Cu at (173.2, 114.9)
- added RpontAlu1: 50, Resistor_THT:R_Axial_DIN0207_L6.3mm_D2.5mm_P10.16mm_Horizontal, F.Cu at (125.0, 108.6)
- added U1: RN2483, MyAIME:RN2483, F.Cu at (159.3, 88.3)
- added U2: LTC1100xN8, Package_DIP:DIP-8_W7.62mm, F.Cu at (147.8, 106.0)
- moved J1 26.2 mm to (125.0, 113.7), turned to 90 degrees
- moved R6 16.3 mm to (117.3, 102.2), turned to 270 degrees
- renumbered R1 to R6
Connections:
- J1 pad 1: /Alu9 -> /PolySi7
- J1 pad 2: GND -> /Vin
- P1 pad 3: /Reset -> ~Reset
- P2 pad 1: /A0 -> A0
- P2 pad 2: /A1 -> Valu
- P4 pad 7: /1(Tx) -> TX
- P4 pad 8: /0(Rx) -> RX
- R6 pad 2: /PolySi2 -> GND
- R6 pad 3: /Gaz3 -> +5V
- R6 pad 4: /Alu4 -> GND
- R6 pad 9: /Alu9 -> Valu

Commit message: Kicad Version2.0
Parts:
- removed the U1 at (159.3, 88.3)
- added J1: Conn_01x08_Female, Connector_PinSocket_2.54mm:PinSocket_1x08_P2.54mm_Vertical, F.Cu at (170.7, 83.2)
- added U2: RN2483_Breakout, MyAIME:SIP-8, F.Cu at (86.9, 90.8)
- C1, C2, C3, C4: footprint Capacitor_THT:C_Radial_D5.0mm_H7.0mm_P2.00mm -> Capacitor_THT:C_Radial_D4.0mm_H5.0mm_P1.50mm
- renumbered J1 to J2, U2 to U1
Routing:
- net +5V: track 0.00 -> 69.3 mm
- net Net-(C3-Pad2): track 0.00 -> 59.3 mm
- net Valu: track 0.00 -> 59.0 mm, vias 0 -> 4
- net Net-(C1-Pad1): track 0.00 -> 53.2 mm, vias 0 -> 1
- net ~Reset: track 0.00 -> 53.0 mm
- net +3V3: track 0.00 -> 45.4 mm
- net /Vin: track 0.00 -> 34.7 mm, vias 0 -> 2
- net A0: track 0.00 -> 28.2 mm
- net Net-(C3-Pad1): track 0.00 -> 27.0 mm
- net /Gaz1: track 0.00 -> 24.4 mm
- net RX: track 0.00 -> 13.2 mm
- net /PolySi7: track 0.00 -> 10.8 mm
- net TX: track 0.00 -> 8.15 mm
- added copper zone on B.Cu, net GND
- added copper zone on F.Cu, net GND
