File: Ana/Ana.sch (KiCad schematic (older format))
At the start: 22 parts, among them J1 Conn_01x02_Female, P1 Power, P2 Analog, P3 Digital, P4 Digital, P5 CONN_01X01, P6 CONN_01X01, P7 CONN_01X01, P8 CONN_01X01, U1 LTC1100xN8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

Commit message: Waiting for PCB layout
Parts:
- C1: footprint (none) -> Capacitor_THT:C_Radial_D4.0mm_H5.0mm_P1.50mm
- C2: renamed from C3; footprint (none) -> Capacitor_THT:C_Radial_D4.0mm_H5.0mm_P1.50mm
- C3: renamed from C4; footprint (none) -> Capacitor_THT:C_Radial_D4.0mm_H5.0mm_P1.50mm
- C4: renamed from C2; footprint (none) -> Capacitor_THT:C_Radial_D4.0mm_H5.0mm_P1.50mm
- R1: renamed from R5; footprint (none) -> Resistor_THT:R_Axial_DIN0207_L6.3mm_D2.5mm_P10.16mm_Horizontal
- R2: renamed from R1; footprint (none) -> Resistor_THT:R_Axial_DIN0207_L6.3mm_D2.5mm_P10.16mm_Horizontal
- R3: renamed from R2; footprint (none) -> Resistor_THT:R_Axial_DIN0207_L6.3mm_D2.5mm_P10.16mm_Horizontal
- R4: renamed from R3; footprint (none) -> Resistor_THT:R_Axial_DIN0207_L6.3mm_D2.5mm_P10.16mm_Horizontal
- R5: renamed from R6; footprint (none) -> Resistor_THT:R_Axial_DIN0207_L6.3mm_D2.5mm_P10.16mm_Horizontal
- RpontAlu1: footprint (none) -> Resistor_THT:R_Axial_DIN0207_L6.3mm_D2.5mm_P10.16mm_Horizontal
- renumbered R1 to R6, U1 to U2
Changed lines of the file:
@@
 ~Reset
 $Comp
-L power:+3.3V #PWR01
+L power:+3.3V #PWR07
 U 1 1 56D70538
 P 9150 1450
-F 0 "#PWR01" H 9150 1300 50  0001 C CNN
+F 0 "#PWR07" H 9150 1300 50  0001 C CNN
 F 1 "+3.3V" V 9150 1700 50  0000 C CNN
 F 2 "" H 9150 1450 50  0000 C CNN
@@
 $EndComp
 $Comp
-L power:+5V #PWR02
+L power:+5V #PWR06
 U 1 1 56D707BB
 P 9050 1350
-F 0 "#PWR02" H 9050 1200 50  0001 C CNN
+F 0 "#PWR06" H 9050 1200 50  0001 C CNN
 F 1 "+5V" V 9050 1550 50  0000 C CNN
 F 2 "" H 9050 1350 50  0000 C CNN
@@
 $EndComp
 $Comp
-L power:GND #PWR03
+L power:GND #PWR08
 U 1 1 56D70CC2
 P 9300 3150
-F 0 "#PWR03" H 9300 2900 50  0001 C CNN
+F 0 "#PWR08" H 9300 2900 50  0001 C CNN
 F 1 "GND" H 9300 3000 50  0000 C CNN
 F 2 "" H 9300 3150 50  0000 C CNN
@@
 $EndComp
 $Comp
-L power:GND #PWR04
+L power:GND #PWR09
 U 1 1 56D70CFF
 P 10300 3150
-F 0 "#PWR04" H 10300 2900 50  0001 C CNN
+F 0 "#PWR09" H 10300 2900 50  0001 C CNN
 F 1 "GND" H 10300 3000 50  0000 C CNN
 F 2 "" H 10300 3150 50  0000 C CNN
@@
 $EndComp
 $Comp
-L aime:AIME R1
+L aime:AIME R6
 U 1 1 5FD1A66A
 P 6450 2150
-F 0 "R1" H 6467 2504 50  0000 C CNN
+F 0 "R6" H 6467 2504 50  0000 C CNN
 F 1 "AIME" H 6467 2413 50  0000 C CNN
 F 2 "MyAIME:TO-5-10_Window" H 6467 2322 50  0000 C CNN
@@
 PolySi2
 $Comp
-L power:GND #PWR06
+L power:GND #PWR03
 U 1 1 5FD2A34A
 P 6800 850
-F 0 "#PWR06" H 6800 600 50  0001 C CNN
+F 0 "#PWR03" H 6800 600 50  0001 C CNN
 F 1 "GND" H 6800 700 50  0000 C CNN
 F 2 "" H 6800 850 50  0000 C CNN
@@
 $EndComp
 $Comp
-L power:+3.3V #PWR07
+L power:+3.3V #PWR04
 U 1 1 5FD2FF65
 P 7300 850
-F 0 "#PWR07" H 7300 700 50  0001 C CNN
+F 0 "#PWR04" H 7300 700 50  0001 C CNN
 F 1 "+3.3V" V 7300 1100 50  0000 C CNN
 F 2 "" H 7300 850 50  0000 C CNN
@@
 F 0 "RpontAlu1" V 7243 2150 50  0000 C CNN
 F 1 "50" V 7334 2150 50  0000 C CNN
-F 2 "" V 7380 2150 50  0001 C CNN
+F 2 "Resistor_THT:R_Axial_DIN0207_L6.3mm_D2.5mm_P10.16mm_Horizontal" V 7380 2150 50  0001 C CNN
 F 3 "~" H 7450 2150 50  0001 C CNN
 	1    7450 2150
@@
 	6700 2300 8100 2300
 $Comp
-L Device:R_US R5
+L Device:R_US R1
 U 1 1 5FD166AE
 P 1100 2300
-F 0 "R5" V 1305 2300 50  0000 C CNN
+F 0 "R1" V 1305 2300 50  0000 C CNN
 F 1 "10k" V 1214 2300 50  0000 C CNN
-F 2 "" V 1140 2290 50  0001 C CNN
+F 2 "Resistor_THT:R_Axial_DIN0207_L6.3mm_D2.5mm_P10.16mm_Horizontal" V 1140 2290 50  0001 C CNN
 F 3 "~" H 1100 2300 50  0001 C CNN
 	1    1100 2300
@@
 $EndComp
 $Comp
-L Device:R_US R1
+L Device:R_US R2
 U 1 1 5FD19DCD
 P 1800 2700
-F 0 "R1" H 1732 2654 50  0000 R CNN
+F 0 "R2" H 1732 2654 50  0000 R CNN
 F 1 "100k" H 1732 2745 50  0000 R CNN
-F 2 "" V 1840 2690 50  0001 C CNN
+F 2 "Resistor_THT:R_Axial_DIN0207_L6.3mm_D2.5mm_P10.16mm_Horizontal" V 1840 2690 50  0001 C CNN
 F 3 "~" H 1800 2700 50  0001 C CNN
 	1    1800 2700
@@
 $EndComp
 $Comp
-L Device:R_US R2
+L Device:R_US R3
 U 1 1 5FD1C98B
 P 2200 2700
-F 0 "R2" H 2132 2654 50  0000 R CNN
+F 0 "R3" H 2132 2654 50  0000 R CNN
 F 1 "1k" H 2132 2745 50  0000 R CNN
-F 2 "" V 2240 2690 50  0001 C CNN
+F 2 "Resistor_THT:R_Axial_DIN0207_L6.3mm_D2.5mm_P10.16mm_Horizontal" V 2240 2690 50  0001 C CNN
 F 3 "~" H 2200 2700 50  0001 C CNN
 	1    2200 2700
@@
 F 0 "C1" H 1365 2746 50  0000 L CNN
 F 1 "100n" H 1365 2655 50  0000 L CNN
-F 2 "" H 1288 2550 50  0001 C CNN
+F 2 "Capacitor_THT:C_Radial_D4.0mm_H5.0mm_P1.50mm" H 1288 2550 50  0001 C CNN
 F 3 "~" H 1250 2700 50  0001 C CNN
 	1    1250 2700
@@
 NoConn ~ 2900 2200
 $Comp
-L Amplifier_Instrumentation:LTC1100xN8 U1
+L Amplifier_Instrumentation:LTC1100xN8 U2
 U 1 1 5FD3211E
 P 2900 1900
-F 0 "U1" H 3244 1854 50  0000 L CNN
+F 0 "U2" H 3244 1854 50  0000 L CNN
 F 1 "LTC1100xN8" H 3244 1945 50  0000 L CNN
 F 2 "Package_DIP:DIP-8_W7.62mm" H 2900 1900 50  0001 C CNN
@@
 $EndComp
 $Comp
-L Device:C C4
+L Device:C C3
 U 1 1 5FD27FBD
 P 3650 1750
-F 0 "C4" H 3765 1796 50  0000 L CNN
+F 0 "C3" H 3765 1796 50  0000 L CNN
 F 1 "1u" H 3765 1705 50  0000 L CNN
-F 2 "" H 3688 1600 50  0001 C CNN
+F 2 "Capacitor_THT:C_Radial_D4.0mm_H5.0mm_P1.50mm" H 3688 1600 50  0001 C CNN
 F 3 "~" H 3650 1750 50  0001 C CNN
 	1    3650 1750
@@
 $EndComp
 $Comp
-L Device:C C3
+L Device:C C2
 U 1 1 5FD269EA
 P 3250 2600
-F 0 "C3" H 3365 2646 50  0000 L CNN
+F 0 "C2" H 3365 2646 50  0000 L CNN
 F 1 "100n" H 3365 2555 50  0000 L CNN
-F 2 "" H 3288 2450 50  0001 C CNN
+F 2 "Capacitor_THT:C_Radial_D4.0mm_H5.0mm_P1.50mm" H 3288 2450 50  0001 C CNN
 F 3 "~" H 3250 2600 50  0001 C CNN
 	1    3250 2600
@@
 $EndComp
 $Comp
-L Device:C C2
+L Device:C C4
 U 1 1 5FD25400
 P 4850 2250
-F 0 "C2" H 4965 2296 50  0000 L CNN
+F 0 "C4" H 4965 2296 50  0000 L CNN
 F 1 "100n" H 4965 2205 50  0000 L CNN
-F 2 "" H 4888 2100 50  0001 C CNN
+F 2 "Capacitor_THT:C_Radial_D4.0mm_H5.0mm_P1.50mm" H 4888 2100 50  0001 C CNN
 F 3 "~" H 4850 2250 50  0001 C CNN
 	1    4850 2250
@@
 $EndComp
 $Comp
-L Device:R_US R6
+L Device:R_US R5
 U 1 1 5FD1F592
 P 4600 1900
-F 0 "R6" V 4395 1900 50  0000 C CNN
+F 0 "R5" V 4395 1900 50  0000 C CNN
 F 1 "1k" V 4486 1900 50  0000 C CNN
-F 2 "" V 4640 1890 50  0001 C CNN
+F 2 "Resistor_THT:R_Axial_DIN0207_L6.3mm_D2.5mm_P10.16mm_Horizontal" V 4640 1890 50  0001 C CNN
 F 3 "~" H 4600 1900 50  0001 C CNN
 	1    4600 1900
@@
 $EndComp
 $Comp
-L Device:R_US R3
+L Device:R_US R4
 U 1 1 5FD1B3AC
 P 4150 1750
-F 0 "R3" H 4218 1796 50  0000 L CNN
+F 0 "R4" H 4218 1796 50  0000 L CNN
 F 1 "100k" H 4218 1705 50  0000 L CNN
-F 2 "" V 4190 1740 50  0001 C CNN
+F 2 "Resistor_THT:R_Axial_DIN0207_L6.3mm_D2.5mm_P10.16mm_Horizontal" V 4190 1740 50  0001 C CNN
 F 3 "~" H 4150 1750 50  0001 C CNN
 	1    4150 1750
@@
 Connection ~ 2200 3000
 $Comp
-L power:GND #PWR0101
+L power:GND #PWR01
 U 1 1 5FD5C1E1
 P 2450 3000
-F 0 "#PWR0101" H 2450 2750 50  0001 C CNN
+F 0 "#PWR01" H 2450 2750 50  0001 C CNN
 F 1 "GND" H 2455 2827 50  0000 C CNN
 F 2 "" H 2450 3000 50  0001 C CNN
@@
 +3.3V
 $Comp
-L power:GND #PWR0102
+L power:GND #PWR02
 U 1 1 5FD6B892
 P 3800 5150
-F 0 "#PWR0102" H 3800 4900 50  0001 C CNN
+F 0 "#PWR02" H 3800 4900 50  0001 C CNN
 F 1 "GND" H 3805 4977 50  0000 C CNN
 F 2 "" H 3800 5150 50  0001 C CNN

Commit message: Kicad Version2.0
Parts:
- removed U1: RN2483, MyAIME:RN2483, symbol rn2483:RN2483
- added J1: Conn_01x08_Female, Connector_PinSocket_2.54mm:PinSocket_1x08_P2.54mm_Vertical, symbol Connector:Conn_01x08_Female
- added U2: RN2483_Breakout, MyAIME:SIP-8, symbol RN2483_Breakout:RN2483_Breakout
- renumbered J1 to J2, U2 to U1
Connections:
- net +3V3: now also J1.6 (Pin_6)
- net GND: now also J1.8 (Pin_8)
- net RX: now also J1.2 (Pin_2)
- net TX: now also J1.1 (Pin_1)
- net ~Reset: now also J1.4 (Pin_4)
- no-connect marks 71 -> 35
Changed lines of the file:
@@
 Title "AIME Smart Sensor"
 Date "2020-12-09"
-Rev "1.0"
+Rev "2.0"
 Comp "INSA Toulouse 5ISS Groupe-2"
 Comment1 "Qiang XU"
@@
 ~Reset
 $Comp
-L power:+3.3V #PWR07
+L power:+3.3V #PWR08
 U 1 1 56D70538
 P 9150 1450
-F 0 "#PWR07" H 9150 1300 50  0001 C CNN
+F 0 "#PWR08" H 9150 1300 50  0001 C CNN
 F 1 "+3.3V" V 9150 1700 50  0000 C CNN
 F 2 "" H 9150 1450 50  0000 C CNN
@@
 $EndComp
 $Comp
-L power:+5V #PWR06
+L power:+5V #PWR07
 U 1 1 56D707BB
 P 9050 1350
-F 0 "#PWR06" H 9050 1200 50  0001 C CNN
+F 0 "#PWR07" H 9050 1200 50  0001 C CNN
 F 1 "+5V" V 9050 1550 50  0000 C CNN
 F 2 "" H 9050 1350 50  0000 C CNN
@@
 $EndComp
 $Comp
-L power:GND #PWR08
+L power:GND #PWR09
 U 1 1 56D70CC2
 P 9300 3150
-F 0 "#PWR08" H 9300 2900 50  0001 C CNN
+F 0 "#PWR09" H 9300 2900 50  0001 C CNN
 F 1 "GND" H 9300 3000 50  0000 C CNN
 F 2 "" H 9300 3150 50  0000 C CNN
@@
 $EndComp
 $Comp
-L power:GND #PWR09
+L power:GND #PWR010
 U 1 1 56D70CFF
 P 10300 3150
-F 0 "#PWR09" H 10300 2900 50  0001 C CNN
+F 0 "#PWR010" H 10300 2900 50  0001 C CNN
 F 1 "GND" H 10300 3000 50  0000 C CNN
 F 2 "" H 10300 3150 50  0000 C CNN
@@
 Wire Wire Line
 	10200 1300 10550 1300
-Wire Wire Line
-	10200 1200 10550 1200
 Wire Wire Line
 	10200 3000 10550 3000
@@
 PolySi2
 $Comp
-L power:GND #PWR03
+L power:GND #PWR04
 U 1 1 5FD2A34A
 P 6800 850
-F 0 "#PWR03" H 6800 600 50  0001 C CNN
+F 0 "#PWR04" H 6800 600 50  0001 C CNN
 F 1 "GND" H 6800 700 50  0000 C CNN
 F 2 "" H 6800 850 50  0000 C CNN
@@
 $EndComp
 $Comp
-L power:+3.3V #PWR04
+L power:+3.3V #PWR05
 U 1 1 5FD2FF65
 P 7300 850
-F 0 "#PWR04" H 7300 700 50  0001 C CNN
+F 0 "#PWR05" H 7300 700 50  0001 C CNN
 F 1 "+3.3V" V 7300 1100 50  0000 C CNN
 F 2 "" H 7300 850 50  0000 C CNN
@@
 $EndComp
 $Comp
-L power:+5V #PWR05
+L power:+5V #PWR06
 U 1 1 5FD2FF6B
 P 7800 850
-F 0 "#PWR05" H 7800 700 50  0001 C CNN
+F 0 "#PWR06" H 7800 700 50  0001 C CNN
 F 1 "+5V" V 7800 1050 50  0000 C CNN
 F 2 "" H 7800 850 50  0000 C CNN
@@
 $EndComp
 $Comp
-L Connector:Conn_01x02_Female J1
+L Connector:Conn_01x02_Female J2
 U 1 1 5FD46AE3
 P 7450 3300
-F 0 "J1" H 7478 3276 50  0000 L CNN
+F 0 "J2" H 7478 3276 50  0000 L CNN
 F 1 "Conn_01x02_Female" H 7478 3185 50  0000 L CNN
 F 2 "Connector_PinSocket_1.27mm:PinSocket_1x02_P1.27mm_Vertical" H 7450 3300 50  0001 C CNN
@@
 NoConn ~ 2900 2200
 $Comp
-L Amplifier_Instrumentation:LTC1100xN8 U2
+L Amplifier_Instrumentation:LTC1100xN8 U1
 U 1 1 5FD3211E
 P 2900 1900
-F 0 "U2" H 3244 1854 50  0000 L CNN
+F 0 "U1" H 3244 1854 50  0000 L CNN
 F 1 "LTC1100xN8" H 3244 1945 50  0000 L CNN
 F 2 "Package_DIP:DIP-8_W7.62mm" H 2900 1900 50  0001 C CNN
@@
 Connection ~ 3250 2450
 NoConn ~ 3000 1600
-NoConn ~ 7700 2450
 Text GLabel 5350 1900 2    50   Input ~ 0
 A0
@@
 Wire Wire Line
 	8100 1350 9050 1350
-Text GLabel 3600 5550 2    50   Input ~ 0
+Text GLabel 6050 4100 0    50   Input ~ 0
 RX
-Text GLabel 3600 5650 2    50   Input ~ 0
+Text GLabel 6050 4000 0    50   Input ~ 0
 TX
-Text GLabel 1800 4650 0    50   Input ~ 0
+Text GLabel 6050 4300 0    50   Input ~ 0
 ~Reset
 Text GLabel 10550 3000 2    50   Input ~ 0
@@
 Text Label 3700 2450 0    50   ~ 0
 +5V
-Text Label 3600 5050 0    50   ~ 0
-+3.3V
-$Comp
-L power:GND #PWR02
+$Comp
+L power:GND #PWR03
 U 1 1 5FD6B892
-P 3800 5150
-F 0 "#PWR02" H 3800 4900 50  0001 C CNN
-F 1 "GND" H 3805 4977 50  0000 C CNN
-F 2 "" H 3800 5150 50  0001 C CNN
-F 3 "" H 3800 5150 50  0001 C CNN
-	1    3800 5150
-	1    0    0    -1
-$EndComp
-Wire Wire Line
-	3600 5150 3800 5150
-$Comp
-L rn2483:RN2483 U1
-U 1 1 5FE478AF
-P 2700 4850
-F 0 "U1" H 2700 3369 60  0000 C CNN
-F 1 "RN2483" H 2700 3263 60  0000 C CNN
-F 2 "MyAIME:RN2483" H 2700 3157 60  0000 C CNN
-F 3 "" H 2800 4150 60  0000 C CNN
-	1    2700 4850
-	1    0    0    -1
-$EndComp
-NoConn ~ 2250 3850
-NoConn ~ 2400 3850
-NoConn ~ 2550 3850
-NoConn ~ 2700 3850
-NoConn ~ 2850 3850
-NoConn ~ 3000 3850
-NoConn ~ 3150 3850
-NoConn ~ 3600 4250
-NoConn ~ 3600 4350
-NoConn ~ 3600 4450
-NoConn ~ 3600 4550
-NoConn ~ 3600 4650
-NoConn ~ 3600 4750
-NoConn ~ 3600 4850
-NoConn ~ 3600 4950
-NoConn ~ 3600 5250
-NoConn ~ 3600 5350
-NoConn ~ 3600 5450
-NoConn ~ 3600 5750
-NoConn ~ 3600 5850
-NoConn ~ 3600 5950
-NoConn ~ 3600 6050
-NoConn ~ 3600 6150
-NoConn ~ 1800 6150
-NoConn ~ 1800 6050
-NoConn ~ 1800 5950
-NoConn ~ 1800 5850
-NoConn ~ 1800 5750
-NoConn ~ 1800 5650
-NoConn ~ 1800 5550
-NoConn ~ 1800 5450
-NoConn ~ 1800 5350
-NoConn ~ 1800 5250
-NoConn ~ 1800 5150
-NoConn ~ 1800 5050
-NoConn ~ 1800 4950
-NoConn ~ 1800 4850
-NoConn ~ 1800 4750
-NoConn ~ 1800 4550
-NoConn ~ 1800 4450
-NoConn ~ 1800 4350
-NoConn ~ 1800 4250
+P 6050 4700
+F 0 "#PWR03" H 6050 4450 50  0001 C CNN
+F 1 "GND" H 6055 4527 50  0000 C CNN
+F 2 "" H 6050 4700 50  0001 C CNN
+F 3 "" H 6050 4700 50  0001 C CNN
+	1    6050 4700
+	1    0    0    -1
+$EndComp
 NoConn ~ 8900 2700
 NoConn ~ 8900 2800
-NoConn ~ 8900 2900
-NoConn ~ 8900 3000
 NoConn ~ 10550 2800
 NoConn ~ 10550 2700
@@
 NoConn ~ 10550 1600
 NoConn ~ 10550 1400
-NoConn ~ 10550 1300
-NoConn ~ 10550 1200
 NoConn ~ 9350 1450
+Wire Wire Line
+	6050 4700 6250 4700
+Wire Wire Line
+	6050 4500 6250 4500
+Wire Wire Line
+	6050 4300 6250 4300
+Wire Wire Line
+	6050 4100 6250 4100
+Wire Wire Line
+	6050 4000 6250 4000
+$Comp
+L Connector:Conn_01x08_Female J1
+U 1 1 5FD2D1AF
+P 6450 4300
+F 0 "J1" H 6050 3550 50  0000 L CNN
+F 1 "Conn_01x08_Female" H 6500 3600 50  0000 R BNN
+F 2 "Connector_PinSocket_2.54mm:PinSocket_1x08_P2.54mm_Vertical" H 6450 4300 50  0001 C CNN
+F 3 "~" H 6450 4300 50  0001 C CNN
+	1    6450 4300
+	1    0    0    -1
+$EndComp
+$Comp
+L RN2483_Breakout:RN2483_Breakout U2
+U 1 1 5FD24A37
+P 7150 4400
+F 0 "U2" V 7004 4978 50  0000 L CNN
+F 1 "RN2483_Breakout" V 7095 4978 50  0000 L CNN
+F 2 "MyAIME:SIP-8" V 7186 4978 50  0000 L CNN
+F 3 "" H 7150 5050 50  0001 C CNN
+	1    7150 4400
+	0    1    1    0
+$EndComp
+NoConn ~ 6250 4200
+NoConn ~ 6250 4400
+NoConn ~ 6250 4600
+NoConn ~ 7100 4000
+NoConn ~ 7100 4100
+NoConn ~ 7100 4200
+NoConn ~ 7100 4300
+NoConn ~ 7100 4400
+NoConn ~ 7100 4500
+NoConn ~ 7100 4600
+NoConn ~ 7100 4700
+Text GLabel 8650 1800 0    50   Input ~ 0
+~Reset
+$Comp
+L power:+3.3V #PWR02
+U 1 1 5FD8F9CE
+P 6050 4500
+F 0 "#PWR02" H 6050 4350 50  0001 C CNN
+F 1 "+3.3V" V 6065 4628 50  0000 L CNN
+F 2 "" H 6050 4500 50  0001 C CNN
+F 3 "" H 6050 4500 50  0001 C CNN
+	1    6050 4500
+	0    -1   -1   0
+$EndComp
+Text GLabel 8900 2500 0    50   Input ~ 0
+A0
+Wire Wire Line
+	10200 1200 10550 1200
 $EndSCHEMATC
